Commit message: lua-launch modify

File: src/myrobot_description/xacro/my_robot.xacro (robot description, xacro)
@@ -1,5 +1,4 @@
 <robot name="my_robot" xmlns:xacro="http://wiki.ros.org/xacro">
     <xacro:include filename="my_robot_base.xacro" />
-    <xacro:include filename="my_robot_camera.xacro" />
     <xacro:include filename="my_robot_laser.xacro" />
 </robot>

File: src/myrobot_description/xacro/my_robot_laser.xacro (robot description, xacro)
@@ -6,5 +6,5 @@
     <xacro:property name="laser_length" value="0.02" />
     <xacro:property name="joint_support_x" value="0" />
-    <xacro:property name="joint_support_y" value="0" />
+    <xacro:property name="joint_support_y" value="0.12" />
     <xacro:property name="joint_support_z" value="${base_length / 2 + support_length / 2}" />
     <xacro:property name="joint_laser_x" value="0" />
