Commit message: model modify

File: src/myrobot_description/xacro/my_robot_base.xacro (robot description, xacro)
@@ -99,3 +99,25 @@
     <xacro:wheel_func wheel_name="left" flag="1" />
     <xacro:wheel_func wheel_name="right" flag="-1" />
+    <xacro:property name="small_wheel_radius" value="0.0075" />
+    <xacro:macro name="small_wheel_func" params="small_wheel_name flag">
+        <link name="${small_wheel_name}_wheel">
+            <visual>
+                <geometry>
+                    <sphere radius="${small_wheel_radius}" />
+                </geometry>
+                <origin xyz="0 0 0" rpy="0 0 0" />
+                <material name="wheel_color">
+                    <color rgba="0 0 0 0.8" />
+                </material>
+            </visual>
+        </link>
+        <joint name="${small_wheel_name}2link" type="continuous">
+            <parent link="base_link"  />
+            <child link="${small_wheel_name}_wheel" />
+            <origin xyz="${0.1 * flag} 0 ${-base_h/2}" rpy="0 0 0" />
+            <axis xyz="0 1 0" />
+        </joint>
+    </xacro:macro >
+    <xacro:small_wheel_func small_wheel_name="front" flag="1"/>
+    <xacro:small_wheel_func small_wheel_name="back" flag="-1"/>
 </robot>

Commit message: tf modify

File: src/myrobot_description/xacro/my_robot_base.xacro (robot description, xacro)
@@ -20,6 +20,6 @@
     <xacro:property name="wheel_joint_y" value="0.1515"/>
     <xacro:property name="wheel_joint_z" value="0.00"/>
-    <xacro:property name="base_a" value="0.47"/>
-    <xacro:property name="base_b" value="0.374"/>
+    <xacro:property name="base_a" value="0.374"/>
+    <xacro:property name="base_b" value="0.47"/>
     <xacro:property name="base_h" value="0.264"/>
     <xacro:macro name="cylinder_inertial_matrix" params="m r h">

File: src/myrobot_description/xacro/my_robot_laser.xacro (robot description, xacro)
@@ -5,6 +5,6 @@
     <xacro:property name="laser_radius" value="0.03" />
     <xacro:property name="laser_length" value="0.02" />
-    <xacro:property name="joint_support_x" value="0" />
-    <xacro:property name="joint_support_y" value="0.12" />
+    <xacro:property name="joint_support_x" value="0.12" />
+    <xacro:property name="joint_support_y" value="0" />
     <xacro:property name="joint_support_z" value="${base_length / 2 + support_length / 2}" />
     <xacro:property name="joint_laser_x" value="0" />
@@ -39,5 +39,5 @@
         <parent link="support" />
         <child link="laser"/>
-        <origin xyz="${joint_laser_x} ${joint_laser_y} ${joint_laser_z}" rpy="0 0 0" />
+        <origin xyz="${joint_laser_x} ${joint_laser_y} ${joint_laser_z}" rpy="0 0 -1.57" />
     </joint>
 </robot>
